Commit message: robots! (pr2 drake, panda drake, panda pb but with sphere collisions)

File: models/panda/robots/panda_arm_hand.urdf (robot description, URDF)
Before this commit: robot panda, 14 links, 13 joints
Joints:
- joint camera_frame_joint: origin xyz=0.030768772587180138, 0.0, 0.05 rpy=0 0 -1.5708 -> xyz=0.030768772587180138 0.0 0.05 rpy=0 0 -1.5708
