Commit message: updated drake movo model

File: models/movo_drake/movo_robotiq_collision.urdf (robot description, URDF)
Before this commit: robot movo, 58 links, 57 joints
Links:
- link base_chassis_link: geometry collision mesh filename=package://movo_description_drake/meshes/movo_components/col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; visual mesh filename=package://movo_description_drake/meshes/movo_components/col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
- link kinect2_link: geometry collision mesh filename=package://movo_description_drake/meshes/sensors/collision/k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; visual mesh filename=package://movo_description_drake/meshes/sensors/collision/k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
- link left_arm_half_1_link: geometry collision mesh filename=package://movo_description_drake/meshes/manipulation/jaco/c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; visual mesh filename=package://movo_description_drake/meshes/manipulation/jaco/c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
- link left_arm_half_2_link: geometry collision mesh filename=package://movo_description_drake/meshes/manipulation/jaco/c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; visual mesh filename=package://movo_description_drake/meshes/manipulation/jaco/c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
- link left_base_link: geometry collision mesh filename=package://movo_description_drake/meshes/manipulation/jaco/c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; visual mesh filename=package://movo_description_drake/meshes/manipulation/jaco/c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
- link left_forearm_link: geometry collision mesh filename=package://movo_description_drake/meshes/manipulation/jaco/c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; visual mesh filename=package://movo_description_drake/meshes/manipulation/jaco/c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
- link left_gripper_base_link: geometry collision mesh filename=package://movo_description_drake/meshes/manipulation/kinova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; visual mesh filename=package://movo_description_drake/meshes/manipulation/kinova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
- link left_gripper_finger1_finger_tip_link: geometry collision mesh filename=package://movo_description_drake/meshes/manipulation/kinova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; visual mesh filename=package://movo_description_drake/meshes/manipulation/kinova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
- link left_gripper_finger1_knuckle_link: geometry collision mesh filename=package://movo_description_drake/meshes/manipulation/kinova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; visual mesh filename=package://movo_description_drake/meshes/manipulation/kinova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
- link left_gripper_finger2_finger_tip_link: geometry collision mesh filename=package://movo_description_drake/meshes/manipulation/kinova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; visual mesh filename=package://movo_description_drake/meshes/manipulation/kinova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
- link left_gripper_finger2_knuckle_link: geometry collision mesh filename=package://movo_description_drake/meshes/manipulation/kinova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; visual mesh filename=package://movo_description_drake/meshes/manipulation/kinova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
- link left_gripper_finger3_finger_tip_link: geometry collision mesh filename=package://movo_description_drake/meshes/manipulation/kinova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; visual mesh filename=package://movo_description_drake/meshes/manipulation/kinova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
- link left_gripper_finger3_knuckle_link: geometry collision mesh filename=package://movo_description_drake/meshes/manipulation/kinova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; visual mesh filename=package://movo_description_drake/meshes/manipulation/kinova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
- link left_shoulder_link: geometry collision mesh filename=package://movo_description_drake/meshes/manipulation/jaco/c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; visual mesh filename=package://movo_description_drake/meshes/manipulation/jaco/c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
- link left_wrist_3_link: geometry collision mesh filename=package://movo_description_drake/meshes/manipulation/jaco/c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; visual mesh filename=package://movo_description_drake/meshes/manipulation/jaco/c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
- link left_wrist_spherical_1_link: geometry collision mesh filename=package://movo_description_drake/meshes/manipulation/jaco/c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; visual mesh filename=package://movo_description_drake/meshes/manipulation/jaco/c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
- link left_wrist_spherical_2_link: geometry collision mesh filename=package://movo_description_drake/meshes/manipulation/jaco/c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; visual mesh filename=package://movo_description_drake/meshes/manipulation/jaco/c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
- link linear_actuator_fixed_link: geometry collision mesh filename=package://movo_description_drake/meshes/movo_components/col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; visual mesh filename=package://movo_description_drake/meshes/movo_components/col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
- link linear_actuator_link: geometry collision mesh filename=package://movo_description_drake/meshes/movo_components/col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; visual mesh filename=package://movo_description_drake/meshes/movo_components/col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
- link lower_body_link: geometry visual mesh filename=package://movo_description_drake/meshes/movo_body/movo_lowe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
- link mid_body_link: geometry visual mesh filename=package://movo_description_drake/meshes/movo_body/movo_mid_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
- link pan_base_link: geometry collision mesh filename=package://movo_description_drake/meshes/pan_tilt/collision/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; visual mesh filename=package://movo_description_drake/meshes/pan_tilt/collision/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
- link pan_link: geometry collision mesh filename=package://movo_description_drake/meshes/pan_tilt/collision/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; visual mesh filename=package://movo_description_drake/meshes/pan_tilt/collision/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
- link right_arm_half_1_link: geometry collision mesh filename=package://movo_description_drake/meshes/manipulation/jaco/c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; visual mesh filename=package://movo_description_drake/meshes/manipulation/jaco/c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
- link right_arm_half_2_link: geometry collision mesh filename=package://movo_description_drake/meshes/manipulation/jaco/c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; visual mesh filename=package://movo_description_drake/meshes/manipulation/jaco/c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
- link right_base_link: geometry collision mesh filename=package://movo_description_drake/meshes/manipulation/jaco/c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; visual mesh filename=package://movo_description_drake/meshes/manipulation/jaco/c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
- link right_forearm_link: geometry collision mesh filename=package://movo_description_drake/meshes/manipulation/jaco/c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; visual mesh filename=package://movo_description_drake/meshes/manipulation/jaco/c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
- link right_gripper_base_link: geometry collision mesh filename=package://movo_description_drake/meshes/manipulation/roboti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; visual mesh filename=package://movo_description_drake/meshes/manipulation/roboti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
- link right_gripper_finger1_finger_link: geometry collision mesh filename=package://movo_description_drake/meshes/manipulation/roboti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; visual mesh filename=package://movo_description_drake/meshes/manipulation/roboti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
- link right_gripper_finger1_finger_tip_link: geometry collision mesh filename=package://movo_description_drake/meshes/manipulation/roboti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; visual mesh filename=package://movo_description_drake/meshes/manipulation/roboti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
- link right_gripper_finger1_inner_knuckle_link: geometry collision mesh filename=package://movo_description_drake/meshes/manipulation/roboti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; visual mesh filename=package://movo_description_drake/meshes/manipulation/roboti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
- link right_gripper_finger1_knuckle_link: geometry collision mesh filename=package://movo_description_drake/meshes/manipulation/roboti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; visual mesh filename=package://movo_description_drake/meshes/manipulation/roboti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
- link right_gripper_finger2_finger_link: geometry collision mesh filename=package://movo_description_drake/meshes/manipulation/roboti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; visual mesh filename=package://movo_description_drake/meshes/manipulation/roboti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
- link right_gripper_finger2_finger_tip_link: geometry collision mesh filename=package://movo_description_drake/meshes/manipulation/roboti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; visual mesh filename=package://movo_description_drake/meshes/manipulation/roboti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
- link right_gripper_finger2_inner_knuckle_link: geometry collision mesh filename=package://movo_description_drake/meshes/manipulation/roboti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; visual mesh filename=package://movo_description_drake/meshes/manipulation/roboti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
- link right_gripper_finger2_knuckle_link: geometry collision mesh filename=package://movo_description_drake/meshes/manipulation/roboti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; visual mesh filename=package://movo_description_drake/meshes/manipulation/roboti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
- link right_robotiq_coupler_link: geometry collision mesh filename=package://movo_description_drake/meshes/manipulation/roboti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; visual mesh filename=package://movo_description_drake/meshes/manipulation/roboti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
- link right_shoulder_link: geometry collision mesh filename=package://movo_description_drake/meshes/manipulation/jaco/c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; visual mesh filename=package://movo_description_drake/meshes/manipulation/jaco/c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
- link right_wrist_3_link: geometry collision mesh filename=package://movo_description_drake/meshes/manipulation/jaco/c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; visual mesh filename=package://movo_description_drake/meshes/manipulation/jaco/c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
- link right_wrist_spherical_1_link: geometry collision mesh filename=package://movo_description_drake/meshes/manipulation/jaco/c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; visual mesh filename=package://movo_description_drake/meshes/manipulation/jaco/c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
- link right_wrist_spherical_2_link: geometry collision mesh filename=package://movo_description_drake/meshes/manipulation/jaco/c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; visual mesh filename=package://movo_description_drake/meshes/manipulation/jaco/c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
- link tilt_link: geometry collision mesh filename=package://movo_description_drake/meshes/pan_tilt/collision/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; visual mesh filename=package://movo_description_drake/meshes/pan_tilt/collision/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
- link upper_body_link: geometry visual mesh filename=package://movo_description_drake/meshes/movo_body/movo_uppe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
